File: Hardware/BigTime45.brd (EAGLE design)
At the start: 25.1 x 25.1 mm, 18 parts, among them J1 AVR_SPI_PRG_6TESTPOINTS-SM, U2 ATMEGA328P_TQFP, Y1 32.768kHz

Commit message: reposition disp button pad
Parts:
- moved TP3 1.14 mm to (24.3, 24.6)
Routing:
- net BTN: track 25.2 -> 24.5 mm
Changed lines of the file:
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@@
 <setting verticaltext="up"/>
 </settings>
-<grid distance="0.025" unitdist="inch" unit="inch" style="lines" multiple="1" display="yes" altdistance="0.00125" altunitdist="inch" altunit="inch"/>
+<grid distance="0.025" unitdist="inch" unit="inch" style="lines" multiple="1" display="yes" altdistance="0.00625" altunitdist="inch" altunit="inch"/>
 <layers>
 <layer number="1" name="Top" color="4" fill="1" visible="yes" active="yes"/>
@@
 <attribute name="VALUE" x="14.097" y="17.399" size="0.0254" layer="28" rot="MR0"/>
 </element>
-<element name="TP3" library="SparkFun-Connectors" package="1X01_2MM" value="" x="23.33625" y="25.24125"/>
+<element name="TP3" library="SparkFun-Connectors" package="1X01_2MM" value="" x="24.28875" y="24.60625"/>
 <element name="TP4" library="SparkFun-Connectors" package="1X01_2MM" value="" x="26.416" y="16.51"/>
 <element name="TP5" library="adafruit" package="1X01-CLEANBIG" value="" x="6.985" y="8.89" smashed="yes">
@@
 <contactref element="TP3" pad="1"/>
 <wire x1="24.13" y1="13.1445" x2="24.13" y2="21.59" width="0.1524" layer="16"/>
-<wire x1="24.13" y1="21.59" x2="22.225" y2="23.495" width="0.1524" layer="16"/>
-<wire x1="22.225" y1="23.495" x2="22.225" y2="24.13" width="0.1524" layer="16"/>
-<wire x1="22.225" y1="24.13" x2="23.33625" y2="25.24125" width="0.1524" layer="16"/>
 <wire x1="17.405" y1="5.2959" x2="17.405" y2="6.05825" width="0.1524" layer="1"/>
 <wire x1="17.405" y1="6.05825" x2="16.9545" y2="6.50875" width="0.1524" layer="1"/>
@@
 <wire x1="17.399" y1="7.90575" x2="16.9545" y2="7.46125" width="0.1524" layer="16"/>
 <wire x1="16.9545" y1="7.46125" x2="16.9545" y2="6.50875" width="0.1524" layer="16"/>
+<wire x1="24.28875" y1="24.60625" x2="22.86" y2="23.1775" width="0.1524" layer="16"/>
+<wire x1="22.86" y1="23.1775" x2="22.86" y2="22.86" width="0.1524" layer="16"/>
+<wire x1="22.86" y1="22.86" x2="24.13" y2="21.59" width="0.1524" layer="16"/>
 </signal>
 <signal name="SET">

Commit message: more button work
Parts:
- TP3, TP4: device SparkFun-Connectors:1X01_2MM -> Connectors:WATCHBTN
- moved TP3 0.45 mm to (24.6, 24.9), turned to 40 degrees
- moved TP4 0.16 mm to (26.3, 16.5)
Routing:
- net BTN: track 24.5 -> 23.9 mm
Changed lines of the file:
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@@
 <wire x1="6.35" y1="8.255" x2="5.08" y2="6.985" width="0.1524" layer="51"/>
 <wire x1="22.86" y1="8.255" x2="24.13" y2="6.985" width="0.1524" layer="51"/>
+<rectangle x1="25.87625" y1="15.08125" x2="27.14625" y2="17.93875" layer="16"/>
 </plain>
 <attributes>
@@
 <attribute name="VALUE" x="14.097" y="17.399" size="0.0254" layer="28" rot="MR0"/>
 </element>
-<element name="TP3" library="SparkFun-Connectors" package="1X01_2MM" value="" x="24.28875" y="24.60625"/>
-<element name="TP4" library="SparkFun-Connectors" package="1X01_2MM" value="" x="26.416" y="16.51"/>
+<element name="TP3" library="Connectors" package="WATCHBTN" value="" x="24.60625" y="24.92375" rot="R40"/>
+<element name="TP4" library="Connectors" package="WATCHBTN" value="" x="26.25725" y="16.51" smashed="yes">
+<attribute name="NAME" x="24.91105" y="18.3388" size="1.27" layer="25"/>
+<attribute name="VALUE" x="24.98725" y="13.335" size="1.27" layer="27"/>
+</element>
 <element name="TP5" library="adafruit" package="1X01-CLEANBIG" value="" x="6.985" y="8.89" smashed="yes">
 <attribute name="VALUE" x="5.715" y="5.715" size="1.27" layer="27"/>
@@
 <contactref element="U2" pad="32"/>
 <via x="16.9545" y="6.50875" extent="1-16" drill="0.3302"/>
-<wire x1="24.13" y1="13.1445" x2="18.89125" y2="7.90575" width="0.1524" layer="16"/>
+<wire x1="23.65375" y1="12.66825" x2="18.89125" y2="7.90575" width="0.1524" layer="16"/>
 <contactref element="TP3" pad="1"/>
-<wire x1="24.13" y1="13.1445" x2="24.13" y2="21.59" width="0.1524" layer="16"/>
+<wire x1="23.65375" y1="12.66825" x2="23.65375" y2="23.97125" width="0.1524" layer="16"/>
 <wire x1="17.405" y1="5.2959" x2="17.405" y2="6.05825" width="0.1524" layer="1"/>
 <wire x1="17.405" y1="6.05825" x2="16.9545" y2="6.50875" width="0.1524" layer="1"/>
@@
 <wire x1="17.399" y1="7.90575" x2="16.9545" y2="7.46125" width="0.1524" layer="16"/>
 <wire x1="16.9545" y1="7.46125" x2="16.9545" y2="6.50875" width="0.1524" layer="16"/>
-<wire x1="24.28875" y1="24.60625" x2="22.86" y2="23.1775" width="0.1524" layer="16"/>
-<wire x1="22.86" y1="23.1775" x2="22.86" y2="22.86" width="0.1524" layer="16"/>
-<wire x1="22.86" y1="22.86" x2="24.13" y2="21.59" width="0.1524" layer="16"/>
+<wire x1="24.60625" y1="24.92375" x2="23.65375" y2="23.97125" width="0.1524" layer="16"/>
 </signal>
 <signal name="SET">
 <contactref element="U2" pad="1"/>
 <via x="17.6784" y="7.239" extent="1-16" drill="0.3302"/>
-<wire x1="18.669" y1="7.239" x2="25.4" y2="13.97" width="0.1524" layer="16"/>
+<wire x1="18.669" y1="7.239" x2="26.25725" y2="14.82725" width="0.1524" layer="16"/>
 <contactref element="TP4" pad="1"/>
-<wire x1="25.4" y1="13.97" x2="25.4" y2="15.875" width="0.1524" layer="16"/>
-<wire x1="25.4" y1="15.875" x2="26.035" y2="16.51" width="0.1524" layer="16"/>
-<wire x1="26.035" y1="16.51" x2="26.416" y2="16.51" width="0.1524" layer="16"/>
 <wire x1="18.8976" y1="6.7885" x2="18.1289" y2="6.7885" width="0.1524" layer="1"/>
 <wire x1="18.1289" y1="6.7885" x2="17.6784" y2="7.239" width="0.1524" layer="1"/>
 <wire x1="18.669" y1="7.239" x2="17.6784" y2="7.239" width="0.1524" layer="16"/>
+<wire x1="26.25725" y1="16.51" x2="26.25725" y2="14.82725" width="0.1524" layer="16"/>
 </signal>
 <signal name="N$4">
@@
 <vertex x="16.256" y="8.509"/>
 <vertex x="19.05" y="9.525"/>
-<vertex x="22.225" y="12.7"/>
-<vertex x="23.495" y="15.875"/>
-<vertex x="27.94" y="15.875"/>
+<vertex x="21.74875" y="12.3825"/>
+<vertex x="26.82875" y="12.3825"/>
 <vertex x="26.67" y="10.795"/>
 <vertex x="24.13" y="6.985"/>
