File: Hardware/BigTime45.sch (EAGLE design)
At the start: 18 parts, among them J1 AVR_SPI_PRG_6TESTPOINTS-SM, U2 ATMEGA328P_TQFP, Y1 32.768kHz

Commit message: routing
Connections:
- net A: now also U2.ADC7; no longer U2.ADC6
- net B: now also U2.ADC6; no longer J1.1, U2.PB3(MOSI/OC2)
- net C: now also J1.1, U2.PB4(MISO); no longer U2.PB5(SCK)
- net D: now also U2.PB1(OC1A)
- net DIG2: now also J1.4, U2.PB3(MOSI/OC2); no longer U2.PB1(OC1A)
- net DIG3: now also U2.PB0(ICP); no longer J1.3, U2.PB4(MISO)
- net DIG4: now also U2.PD6(AIN0); no longer U2.PD5(T1), U2.PD7(AIN1)
- net DP: now also U2.PD5(T1); no longer J1.4, U2.PB2(SS/OC1B)
- net E: now also J1.3, U2.PB5(SCK); no longer U2.ADC7
- net F: now also U2.PB2(SS/OC1B); no longer U2.PB0(ICP)
- net G: now also U2.PD7(AIN1); no longer U2.PD6(AIN0)
- net N$1: now also Y1.1; no longer Y1.2
- net N$2: now also Y1.2; no longer Y1.1
Other:
- moved on the sheet: Y1

Commit message: routing
Parts:
- TP3, TP4: device SparkFun-Connectors:M01PTH -> SparkFun-Connectors:M01PTH_2MM
Connections:
- net A: now also U2.PB5(SCK); no longer U2.ADC7
- net B: now also U2.ADC7; no longer U2.ADC6
- net DIG1: now also U2.ADC6; no longer U2.PC0(ADC0)
- net E: now also U2.PC0(ADC0); no longer U2.PB5(SCK)

Commit message: tweak
Connections:
- net A: now also J1.3
- net E: no longer J1.3
Changed lines of the file:
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@@
 <pinref part="U2" gate="U$1" pin="PB5(SCK)"/>
+</segment>
+<segment>
+<pinref part="J1" gate="G$1" pin="3"/>
+<wire x1="45.72" y1="149.86" x2="53.34" y2="149.86" width="0.1524" layer="91"/>
 </segment>
 </net>
@@
 </segment>
 <segment>
-<pinref part="J1" gate="G$1" pin="3"/>
-<wire x1="45.72" y1="149.86" x2="53.34" y2="149.86" width="0.1524" layer="91"/>
-</segment>
-<segment>

Commit message: change to 0805 capacitor
Parts:
- C2: device resistor:C-EUC0402 -> resistor:C-EUC0805
Changed lines of the file:
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@@
 <part name="GND2" library="SparkFun" deviceset="GND" device=""/>
 <part name="P+1" library="SparkFun" deviceset="VCC" device=""/>
-<part name="C2" library="resistor" deviceset="C-EU" device="C0402" value="100nF"/>
+<part name="C2" library="resistor" deviceset="C-EU" device="C0805" value="100nF"/>
 <part name="Y1" library="BigTime" deviceset="CRYSTAL" device="TC26H" value="32.768kHz"/>
 <part name="P+4" library="SparkFun" deviceset="VCC" device=""/>

Commit message: more button work
Parts:
- TP3, TP4: device SparkFun-Connectors:M01PTH_2MM -> Connectors:M01EDGE_CONTACT
Changed lines of the file:
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@@
 <part name="BAT+" library="testpad" deviceset="TP" device="TP20R"/>
 <part name="GND1" library="SparkFun" deviceset="GND" device=""/>
-<part name="TP3" library="SparkFun-Connectors" deviceset="M01" device="PTH_2MM"/>
-<part name="TP4" library="SparkFun-Connectors" deviceset="M01" device="PTH_2MM"/>
+<part name="TP3" library="Connectors" deviceset="M01" device="EDGE_CONTACT"/>
+<part name="TP4" library="Connectors" deviceset="M01" device="EDGE_CONTACT"/>
 <part name="TP5" library="adafruit" deviceset="PINHD-1X1" device="CB"/>
 <part name="TP6" library="adafruit" deviceset="PINHD-1X1" device="CB"/>
